File: hardware/rbtnk_bsp.brd (EAGLE design)
At the start: 114 x 80 mm, 20 parts

Commit message: edits eagle layouts
Parts:
- moved R1 51.1 mm to (54.6, 66.0), flipped to the bottom
- moved U$11 48.3 mm to (7.62, 71.1)
- moved U$12 48.3 mm to (20.3, 71.1)
- moved U$13 48.3 mm to (33.0, 71.1)
- moved U$14 48.3 mm to (45.7, 71.1)
- moved U$15 48.3 mm to (58.4, 71.1)
- moved U$16 48.3 mm to (71.1, 71.1)
- moved U$17 48.3 mm to (83.8, 71.1)
- moved U$18 48.3 mm to (96.5, 71.1)
- moved R2 44.4 mm to (54.6, 69.8), flipped to the bottom
- moved U$1 24.4 mm to (7.62, 66.0), flipped to the bottom, turned to 0 degrees
- moved U$2 23.4 mm to (53.3, 63.5), flipped to the bottom, turned to 270 degrees
- moved U$10 2.54 mm to (96.5, 62.2)
- moved U$3 2.54 mm to (7.62, 62.2)
- moved U$4 2.54 mm to (20.3, 62.2)
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Routing:
- net GND: track 235.5 -> 169.0 mm
- net N$18: track 17.1 -> 58.2 mm
- net N$2: track 44.1 -> 13.0 mm
- net N$16: track 30.8 -> 4.21 mm
- net N$19: track 30.7 -> 10.1 mm
- net N$9: track 17.7 -> 37.9 mm
- net N$13: track 32.1 -> 12.9 mm
- net N$10: track 17.6 -> 35.8 mm, vias 0 -> 1
- net N$1: track 52.2 -> 34.3 mm
- net N$14: track 30.4 -> 13.1 mm
- net N$15: track 50.6 -> 33.3 mm
- net N$3: track 32.4 -> 16.0 mm, vias 1 -> 0
- net N$8: track 37.9 -> 53.4 mm
- net N$17: track 26.7 -> 41.9 mm
- net N$4: track 21.8 -> 9.86 mm
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